Commit message: FEAT: add new config

File: ros2_ws/src/diff_drive_hardware/config/diffbot_description.xacro (robot description, xacro)
@@ -19,4 +19,18 @@
       <mass value="1.0"/>
       <inertia ixx="0.0166667" ixy="0" ixz="0" iyy="0.0166667" iyz="0" izz="0.0166667"/>
+    </inertial>
+  </link>
+  <link name="imu_link">
+    <visual>
+      <geometry>
+        <box size="0.04 0.04 0.02"/>
+      </geometry>
+      <material name="orange">
+        <color rgba="1 0.5 0 1"/>
+      </material>
+    </visual>
+    <inertial>
+      <mass value="0.01"/>
+      <inertia ixx="1e-6" ixy="0" ixz="0" iyy="1e-6" iyz="0" izz="1e-6"/>
     </inertial>
   </link>
@@ -75,3 +89,8 @@
     <axis xyz="0 0 1"/>
   </joint>
+  <joint name="imu_joint" type="fixed">
+    <parent link="base_link"/>
+    <child link="imu_link"/>
+    <origin xyz="0.05 0 0.15" rpy="0 0 0"/>
+  </joint>
 </robot>

Commit message: FEAT: add laser link

File: ros2_ws/src/diff_drive_hardware/config/diffbot_description.xacro (robot description, xacro)
@@ -94,3 +94,29 @@
     <origin xyz="0.05 0 0.15" rpy="0 0 0"/>
   </joint>
+  <!-- Laser Scanner Sensor -->
+  <link name="sensor_frame">
+    <visual>
+      <geometry>
+        <!-- A simple cylinder representation; customize as needed -->
+        <cylinder radius="0.01" length="0.02"/>
+      </geometry>
+      <material name="red">
+        <color rgba="1 0 0 1"/>
+      </material>
+    </visual>
+    <collision>
+      <geometry>
+        <cylinder radius="0.01" length="0.02"/>
+      </geometry>
+    </collision>
+    <inertial>
+      <mass value="0.05"/>
+      <inertia ixx="0.0001" ixy="0" ixz="0" iyy="0.0001" iyz="0" izz="0.0001"/>
+    </inertial>
+  </link>
+  <joint name="sensor_joint" type="fixed">
+    <parent link="base_link"/>
+    <child link="sensor_frame"/>
+    <origin xyz="0.4 0 0.245" rpy="0 0 0"/>
+  </joint>
 </robot>

Commit message: Add real sizes

File: ros2_ws/src/diff_drive_hardware/config/diffbot_description.xacro (robot description, xacro)
@@ -39,5 +39,5 @@
     <visual>
       <geometry>
-        <cylinder radius="0.033" length="0.02"/>
+        <cylinder radius="0.0925" length="0.02"/>
       </geometry>
       <material name="black">
@@ -47,5 +47,5 @@
     <collision>
       <geometry>
-        <cylinder radius="0.033" length="0.02"/>
+        <cylinder radius="0.0925" length="0.02"/>
       </geometry>
     </collision>
@@ -59,5 +59,5 @@
     <visual>
       <geometry>
-        <cylinder radius="0.033" length="0.02"/>
+        <cylinder radius="0.0925" length="0.02"/>
       </geometry>
       <material name="black">
@@ -67,5 +67,5 @@
     <collision>
       <geometry>
-        <cylinder radius="0.033" length="0.02"/>
+        <cylinder radius="0.0925" length="0.02"/>
       </geometry>
     </collision>
@@ -79,5 +79,5 @@
     <parent link="base_link"/>
     <child link="left_wheel"/>
-    <origin xyz="0 0.085 -0.033" rpy="-1.5707 0 0"/>
+    <origin xyz="0 0.1475 -0.0925" rpy="-1.5707 0 0"/>
     <axis xyz="0 0 1"/>
   </joint>
@@ -86,5 +86,5 @@
     <parent link="base_link"/>
     <child link="right_wheel"/>
-    <origin xyz="0 -0.085 -0.033" rpy="-1.5707 0 0"/>
+    <origin xyz="0 -0.1475 -0.0925" rpy="-1.5707 0 0"/>
     <axis xyz="0 0 1"/>
   </joint>
@@ -92,5 +92,5 @@
     <parent link="base_link"/>
     <child link="imu_link"/>
-    <origin xyz="0.05 0 0.15" rpy="0 0 0"/>
+    <origin xyz="0.4 0 0.245" rpy="0 0 0"/>
   </joint>
   <!-- Laser Scanner Sensor -->

Commit message: feat(lidar): :sparkles: add lidar integration and launch file
- Updated diffbot_description.xacro for lidar joint and link
- Created lidar.dockerfile for lidar setup
- Added stl27l.launch.py for lidar node configuration

File: ros2_ws/src/diff_drive_hardware/config/diffbot_description.xacro (robot description, xacro)
@@ -79,5 +79,5 @@
     <parent link="base_link"/>
     <child link="left_wheel"/>
-    <origin xyz="0 0.1475 -0.0925" rpy="-1.5707 0 0"/>
+    <origin xyz="0 0.1475 -0.0937" rpy="-1.5707 0 0"/>
     <axis xyz="0 0 1"/>
   </joint>
@@ -86,5 +86,5 @@
     <parent link="base_link"/>
     <child link="right_wheel"/>
-    <origin xyz="0 -0.1475 -0.0925" rpy="-1.5707 0 0"/>
+    <origin xyz="0 -0.1475 -0.0937" rpy="-1.5707 0 0"/>
     <axis xyz="0 0 1"/>
   </joint>
@@ -92,5 +92,5 @@
     <parent link="base_link"/>
     <child link="imu_link"/>
-    <origin xyz="0.4 0 0.245" rpy="0 0 0"/>
+    <origin xyz="0.4 0 0.05" rpy="0 0 0"/>
   </joint>
   <!-- Laser Scanner Sensor -->
@@ -120,3 +120,28 @@
     <origin xyz="0.4 0 0.245" rpy="0 0 0"/>
   </joint>
+  <!-- Lidar Link -->
+  <link name="base_laser">
+    <visual>
+      <geometry>
+        <cylinder radius="0.03" length="0.04"/>
+      </geometry>
+      <material name="red">
+        <color rgba="1 0 0 1"/>
+      </material>
+    </visual>
+    <collision>
+      <geometry>
+        <cylinder radius="0.03" length="0.04"/>
+      </geometry>
+    </collision>
+    <inertial>
+      <mass value="0.125"/>
+      <inertia ixx="0.0001" ixy="0" ixz="0" iyy="0.0001" iyz="0" izz="0.0001"/>
+    </inertial>
+  </link>
+  <joint name="lidar_joint" type="fixed">
+    <parent link="base_link"/>
+    <child link="base_laser"/>
+    <origin xyz="0.15 0 0.18" rpy="0 3.14159 -1.5707"/>
+  </joint>
 </robot>

Commit message: Refactor frontier_explorer package into nav2 package
- Updated docker-compose.yml to rename ros2_frontier_explorer service to ros2_nav2 and changed the Dockerfile reference.
- Removed the explore.yaml configuration file and replaced it with a new explore.yaml in the nav2 package.
- Deleted the frontier_explorer package files including __init__.py, launch files, package.xml, setup.cfg, setup.py, and resource files.
- Created a new nav2 package with necessary files including __init__.py, launch files, package.xml, setup.cfg, setup.py, and explore.yaml.
- Updated the ros_node.py in the web_server to remove unused image handling for depth and confidence frames.
- Adjusted the setup configuration for the mower_knife_controller package to correct the install_scripts directive.

File: ros2_ws/src/diff_drive_hardware/config/diffbot_description.xacro (robot description, xacro)
@@ -94,30 +94,4 @@
     <origin xyz="0.4 0 0.05" rpy="0 0 0"/>
   </joint>
-  <!-- Laser Scanner Sensor -->
-  <link name="sensor_frame">
-    <visual>
-      <geometry>
-        <!-- A simple cylinder representation; customize as needed -->
-        <cylinder radius="0.01" length="0.02"/>
-      </geometry>
-      <material name="red">
-        <color rgba="1 0 0 1"/>
-      </material>
-    </visual>
-    <collision>
-      <geometry>
-        <cylinder radius="0.01" length="0.02"/>
-      </geometry>
-    </collision>
-    <inertial>
-      <mass value="0.05"/>
-      <inertia ixx="0.0001" ixy="0" ixz="0" iyy="0.0001" iyz="0" izz="0.0001"/>
-    </inertial>
-  </link>
-  <joint name="sensor_joint" type="fixed">
-    <parent link="base_link"/>
-    <child link="sensor_frame"/>
-    <origin xyz="0.4 0 0.245" rpy="0 0 0"/>
-  </joint>
   <!-- Lidar Link -->
   <link name="base_laser">
@@ -143,5 +117,5 @@
     <parent link="base_link"/>
     <child link="base_laser"/>
-    <origin xyz="0.15 0 0.18" rpy="0 3.14159 -1.5707"/>
+    <origin xyz="0.15 0 0.18" rpy="0 3.14159 -1.59116"/>
   </joint>
 </robot>

Commit message: Add new NAV2 stack implementation (#16)
* feat(lidar): :sparkles: add lidar integration and launch file

- Updated diffbot_description.xacro for lidar joint and link
- Created lidar.dockerfile for lidar setup
- Added stl27l.launch.py for lidar node configuration

* feat(docker): :sparkles: update docker configuration for services

- Added ros2_frontier_explorer and ros2_web_server services
- Updated ros2_slam and ros2_knife_controller configurations
- Improved costmap parameters in explore.yaml for better navigation
- Adjusted scan topics in slam_toolbox_config.yaml for consistency

* chore(ldlidar_stl_ros2): :wrench: update subproject commit to dirty state

* Add ldlidar ROS2 package with network and serial communication support

- Implemented UDP and TCP socket interfaces for Linux in `network_socket_interface_linux.cpp`.
- Developed serial communication interface in `serial_interface_linux.cpp`.
- Created package.xml for the ldlidar ROS2 package, defining dependencies and metadata.
- Added udev rules scripts for device management in `create_udev_rules.sh` and `delete_udev_rules.sh`.
- Defined udev rules in `ldlidar.rules` to remap device serial ports.
- Implemented main application logic in `main.cpp` to handle LiDAR data publishing.

* Refactor frontier_explorer package into nav2 package

- Updated docker-compose.yml to rename ros2_frontier_explorer service to ros2_nav2 and changed the Dockerfile reference.
- Removed the explore.yaml configuration file and replaced it with a new explore.yaml in the nav2 package.
- Deleted the frontier_explorer package files including __init__.py, launch files, package.xml, setup.cfg, setup.py, and resource files.
- Created a new nav2 package with necessary files including __init__.py, launch files, package.xml, setup.cfg, setup.py, and explore.yaml.
- Updated the ros_node.py in the web_server to remove unused image handling for depth and confidence frames.
- Adjusted the setup configuration for the mower_knife_controller package to correct the install_scripts directive.

* refactor(costmap): :recycle: update footprint and parameters

Adjusted global and local costmap footprints for better navigation.
Modified inflation layer parameters and controller settings for improved
performance and responsiveness.

* fix(controller_server): :bug: increase min_theta_velocity_threshold

Adjusted min_theta_velocity_threshold to improve rotation control.
Updated related parameters for better performance and stability.

* feat(controller_server): :sparkles: update controller parameters

Adjusted velocity thresholds and added odometry topic for improved
robot navigation performance. Updated planner and smoother configurations
to enhance path planning and execution.

* fix(costmap): :bug: set min range to zero for obstacle detection

Updated raytrace_min_range and obstacle_min_range to 0.0
to improve obstacle detection capabilities in the costmap.

* fix(costmap): :bug: update inflation radius and turning radius

* fix(planner_server): :bug: disable traveling in unknown space

* fix(costmap): :bug: enable tracking unknown space and adjust ranges

Updated global costmap to track unknown space and increased obstacle
max range. Adjusted inflation parameters for better navigation
performance.

* chore(ldlidar): :wrench: remove obsolete udev rules scripts

Deleted unused scripts for creating and deleting udev rules for ldlidar.
These scripts are no longer necessary for the current implementation.

File: ros2_ws/src/diff_drive_hardware/config/diffbot_description.xacro (robot description, xacro)
@@ -79,5 +79,5 @@
     <parent link="base_link"/>
     <child link="left_wheel"/>
-    <origin xyz="0 0.1475 -0.0925" rpy="-1.5707 0 0"/>
+    <origin xyz="0 0.1475 -0.0937" rpy="-1.5707 0 0"/>
     <axis xyz="0 0 1"/>
   </joint>
@@ -86,5 +86,5 @@
     <parent link="base_link"/>
     <child link="right_wheel"/>
-    <origin xyz="0 -0.1475 -0.0925" rpy="-1.5707 0 0"/>
+    <origin xyz="0 -0.1475 -0.0937" rpy="-1.5707 0 0"/>
     <axis xyz="0 0 1"/>
   </joint>
@@ -92,12 +92,11 @@
     <parent link="base_link"/>
     <child link="imu_link"/>
-    <origin xyz="0.4 0 0.245" rpy="0 0 0"/>
+    <origin xyz="0.4 0 0.05" rpy="0 0 0"/>
   </joint>
-  <!-- Laser Scanner Sensor -->
-  <link name="sensor_frame">
+  <!-- Lidar Link -->
+  <link name="base_laser">
     <visual>
       <geometry>
-        <!-- A simple cylinder representation; customize as needed -->
-        <cylinder radius="0.01" length="0.02"/>
+        <cylinder radius="0.03" length="0.04"/>
       </geometry>
       <material name="red">
@@ -107,16 +106,16 @@
     <collision>
       <geometry>
-        <cylinder radius="0.01" length="0.02"/>
+        <cylinder radius="0.03" length="0.04"/>
       </geometry>
     </collision>
     <inertial>
-      <mass value="0.05"/>
+      <mass value="0.125"/>
       <inertia ixx="0.0001" ixy="0" ixz="0" iyy="0.0001" iyz="0" izz="0.0001"/>
     </inertial>
   </link>
-  <joint name="sensor_joint" type="fixed">
+  <joint name="lidar_joint" type="fixed">
     <parent link="base_link"/>
-    <child link="sensor_frame"/>
-    <origin xyz="0.4 0 0.245" rpy="0 0 0"/>
+    <child link="base_laser"/>
+    <origin xyz="0.15 0 0.18" rpy="0 3.14159 -1.59116"/>
   </joint>
 </robot>

Commit message: refactor: Merge and clear control values instead of assigning them to support libcamera 0.6.0+.

File: ros2_ws/src/diff_drive_hardware/config/diffbot_description.xacro (robot description, xacro)
@@ -1,4 +1,11 @@
 <?xml version="1.0"?>
 <robot xmlns:xacro="http://www.ros.org/wiki/xacro">
+  <!-- Dummy root link (no inertia) to satisfy KDL -->
+  <link name="base_footprint"/>
+  <joint name="base_footprint_joint" type="fixed">
+    <parent link="base_footprint"/>
+    <child link="base_link"/>
+    <origin xyz="0 0 0" rpy="0 0 0"/>
+  </joint>
   <!-- Base Link -->
   <link name="base_link">

Commit message: feat: Integrate AprilTag detection into the camera system, update Docker environment, add camera link to robot description, and remove ROS discovery server variables from RViz start script.

File: ros2_ws/src/diff_drive_hardware/config/diffbot_description.xacro (robot description, xacro)
@@ -126,3 +126,28 @@
     <origin xyz="0.15 0 0.18" rpy="0 3.14159 -1.59116"/>
   </joint>
+  <!-- Camera Link -->
+  <link name="camera">
+    <visual>
+      <geometry>
+        <box size="0.05 0.05 0.05"/>
+      </geometry>
+      <material name="black">
+        <color rgba="0 0 0 1"/>
+      </material>
+    </visual>
+    <collision>
+      <geometry>
+        <box size="0.05 0.05 0.05"/>
+      </geometry>
+    </collision>
+    <inertial>
+      <mass value="0.05"/>
+      <inertia ixx="0.0001" ixy="0" ixz="0" iyy="0.0001" iyz="0" izz="0.0001"/>
+    </inertial>
+  </link>
+  <joint name="camera_joint" type="fixed">
+    <parent link="base_link"/>
+    <child link="camera"/>
+    <origin xyz="0.15 0 0.10" rpy="-1.5707 0 -1.5707"/>
+  </joint>
 </robot>

Commit message: config: Adjust camera joint origin coordinates in diffbot description.

File: ros2_ws/src/diff_drive_hardware/config/diffbot_description.xacro (robot description, xacro)
@@ -149,5 +149,5 @@
     <parent link="base_link"/>
     <child link="camera"/>
-    <origin xyz="0.15 0 0.10" rpy="-1.5707 0 -1.5707"/>
+    <origin xyz="0.45 0 0.10" rpy="-1.5707 0 -1.5500"/>
   </joint>
 </robot>

Commit message: fix: Adjust camera joint origin (xyz and rpy) in diffbot_description.xacro.

File: ros2_ws/src/diff_drive_hardware/config/diffbot_description.xacro (robot description, xacro)
@@ -149,5 +149,5 @@
     <parent link="base_link"/>
     <child link="camera"/>
-    <origin xyz="0.45 0 0.10" rpy="-1.5707 0 -1.5500"/>
+    <origin xyz="0.47 0 0.125" rpy="-1.6100 0 -1.5400"/>
   </joint>
 </robot>

Commit message: Feature/apriltag (#37)
* feat: Integrate AprilTag detection into the camera system, update Docker environment, add camera link to robot description, and remove ROS discovery server variables from RViz start script.

* config: Adjust camera joint origin coordinates in diffbot description.

* fix: Adjust camera joint origin (xyz and rpy) in diffbot_description.xacro.

File: ros2_ws/src/diff_drive_hardware/config/diffbot_description.xacro (robot description, xacro)
@@ -126,3 +126,28 @@
     <origin xyz="0.15 0 0.18" rpy="0 3.14159 -1.59116"/>
   </joint>
+  <!-- Camera Link -->
+  <link name="camera">
+    <visual>
+      <geometry>
+        <box size="0.05 0.05 0.05"/>
+      </geometry>
+      <material name="black">
+        <color rgba="0 0 0 1"/>
+      </material>
+    </visual>
+    <collision>
+      <geometry>
+        <box size="0.05 0.05 0.05"/>
+      </geometry>
+    </collision>
+    <inertial>
+      <mass value="0.05"/>
+      <inertia ixx="0.0001" ixy="0" ixz="0" iyy="0.0001" iyz="0" izz="0.0001"/>
+    </inertial>
+  </link>
+  <joint name="camera_joint" type="fixed">
+    <parent link="base_link"/>
+    <child link="camera"/>
+    <origin xyz="0.47 0 0.125" rpy="-1.6100 0 -1.5400"/>
+  </joint>
 </robot>

Commit message: refactor: Improve frontend ROS and camera stream reliability with auto-reconnect, simplify camera node streaming to be continuous, and add Docker Compose orphan removal."

File: ros2_ws/src/diff_drive_hardware/config/diffbot_description.xacro (robot description, xacro)
@@ -149,5 +149,5 @@
     <parent link="base_link"/>
     <child link="camera"/>
-    <origin xyz="0.47 0 0.125" rpy="-1.6100 0 -1.5400"/>
+    <origin xyz="0.47 0 0.125" rpy="-1.6100 0 -1.5500"/>
   </joint>
 </robot>

Commit message: feat: update diffbot physical dimensions and refine robot_description parameter handling

File: ros2_ws/src/diff_drive_hardware/config/diffbot_description.xacro (robot description, xacro)
@@ -11,6 +11,7 @@
   <link name="base_link">
     <visual>
+      <origin xyz="0.2 0 0" rpy="0 0 0"/>
       <geometry>
-        <box size="0.2 0.3 0.1"/>
+        <box size="0.6 0.3 0.1"/>
       </geometry>
       <material name="blue">
@@ -46,5 +47,5 @@
     <visual>
       <geometry>
-        <cylinder radius="0.0925" length="0.02"/>
+        <cylinder radius="0.0925" length="0.1"/>
       </geometry>
       <material name="black">
