Commit message: chore: update chassis height and wheel dimensions in diffbot description

File: ros2_ws/src/diff_drive_hardware/config/diffbot_description.xacro (robot description, xacro)
@@ -13,5 +13,5 @@
       <origin xyz="0.2 0 0" rpy="0 0 0"/>
       <geometry>
-        <box size="0.6 0.3 0.1"/>
+        <box size="0.6 0.3 0.2"/>
       </geometry>
       <material name="blue">
@@ -47,5 +47,5 @@
     <visual>
       <geometry>
-        <cylinder radius="0.0925" length="0.1"/>
+        <cylinder radius="0.0937" length="0.1"/>
       </geometry>
       <material name="black">
@@ -55,5 +55,5 @@
     <collision>
       <geometry>
-        <cylinder radius="0.0925" length="0.02"/>
+        <cylinder radius="0.0937" length="0.1"/>
       </geometry>
     </collision>
@@ -67,5 +67,5 @@
     <visual>
       <geometry>
-        <cylinder radius="0.0925" length="0.02"/>
+        <cylinder radius="0.0937" length="0.1"/>
       </geometry>
       <material name="black">
@@ -75,5 +75,5 @@
     <collision>
       <geometry>
-        <cylinder radius="0.0925" length="0.02"/>
+        <cylinder radius="0.0937" length="0.1"/>
       </geometry>
     </collision>

Commit message: feat: add Gazebo simulation environment and stack integration for diffbot

File: ros2_ws/src/diff_drive_hardware/config/diffbot_description.xacro (robot description, xacro)
@@ -25,6 +25,7 @@
     </collision>
     <inertial>
-      <mass value="1.0"/>
-      <inertia ixx="0.0166667" ixy="0" ixz="0" iyy="0.0166667" iyz="0" izz="0.0166667"/>
+      <origin xyz="0.18 0.0 -0.02" rpy="0 0 0"/>
+      <mass value="12.0"/>
+      <inertia ixx="0.15" ixy="0" ixz="0" iyy="0.40" iyz="0" izz="0.45"/>
     </inertial>
   </link>

Commit message: refactor: remove base_footprint and cmd_vel relay, configure direct cmd_vel remapping, and update navigation and FastDDS settings

File: ros2_ws/src/diff_drive_hardware/config/diffbot_description.xacro (robot description, xacro)
@@ -1,11 +1,5 @@
 <?xml version="1.0"?>
 <robot xmlns:xacro="http://www.ros.org/wiki/xacro">
-  <!-- Dummy root link (no inertia) to satisfy KDL -->
-  <link name="base_footprint"/>
-  <joint name="base_footprint_joint" type="fixed">
-    <parent link="base_footprint"/>
-    <child link="base_link"/>
-    <origin xyz="0 0 0" rpy="0 0 0"/>
-  </joint>
+  <!-- Base Link (Root Frame) -->
   <!-- Base Link -->
   <link name="base_link">

File: ros2_ws/src/relobot_gazebo/config/diffbot_gazebo_plugins.xacro (robot description, xacro)
@@ -194,6 +194,7 @@
     <plugin filename="gz_ros2_control-system" name="gz_ros2_control::GazeboSimROS2ControlPlugin">
       <parameters>$(find relobot_gazebo)/config/gazebo_controllers.yaml</parameters>
-      <robot_param_node>/robot_state_publisher</robot_param_node>
-      <robot_param>robot_description</robot_param>
+      <ros>
+        <remapping>/diff_drive_controller/cmd_vel_unstamped:=/cmd_vel</remapping>
+      </ros>
     </plugin>
   </gazebo>

Commit message: feat: add Gazebo simulation environment and stack integration for dif… (#81)
* feat: add Gazebo simulation environment and stack integration for diffbot

* chore: add VS Code settings for terminal profiles, shell integration, and consistent LF line endings

* refactor: optimize Nav2 SmacPlanner, add controller spawner watchdog, and improve simulation startup orchestration

* Feat/add new implementation

* fix(gazebo): clean up simulation architecture, fix FastDDS discovery, restore ROS2 control spawner pipeline, and optimize sensors

* fix(docker-compose): default NGINX_TEMPLATE fallback to nginx.sim.conf.template

* refactor: improve explore_lite navigation loop with robust frontier tracking, retries, and timeouts

* refactor: remove base_footprint and cmd_vel relay, configure direct cmd_vel remapping, and update navigation and FastDDS settings

---------

Co-authored-by: glebobos <glebobos>

File: ros2_ws/src/diff_drive_hardware/config/diffbot_description.xacro (robot description, xacro)
@@ -1,11 +1,5 @@
 <?xml version="1.0"?>
 <robot xmlns:xacro="http://www.ros.org/wiki/xacro">
-  <!-- Dummy root link (no inertia) to satisfy KDL -->
-  <link name="base_footprint"/>
-  <joint name="base_footprint_joint" type="fixed">
-    <parent link="base_footprint"/>
-    <child link="base_link"/>
-    <origin xyz="0 0 0" rpy="0 0 0"/>
-  </joint>
+  <!-- Base Link (Root Frame) -->
   <!-- Base Link -->
   <link name="base_link">
@@ -25,6 +19,7 @@
     </collision>
     <inertial>
-      <mass value="1.0"/>
-      <inertia ixx="0.0166667" ixy="0" ixz="0" iyy="0.0166667" iyz="0" izz="0.0166667"/>
+      <origin xyz="0.18 0.0 -0.02" rpy="0 0 0"/>
+      <mass value="12.0"/>
+      <inertia ixx="0.15" ixy="0" ixz="0" iyy="0.40" iyz="0" izz="0.45"/>
     </inertial>
   </link>
